File: DC-Power/DC-Power.kicad_sch (KiCad schematic)
At the start: 0 parts

Commit message: Draw Type-c
Parts:
- added U1: TYPE-C_16PLC-H10_0, JLCImport:TYPE-C_16PLC-H10_0, symbol JLCImport:TYPE-C_16PLC-H10_0
Connections:
- new net +VDC: U1.A4 (VBUS), U1.A9 (VBUS), U1.B4 (VBUS), U1.B9 (VBUS)
- new net CC1: U1.A5 (CC1)
- new net CC2: U1.B5 (CC2)
- new net D+: U1.A6 (D+), U1.B6 (D+)
- new net D-: U1.A7 (D-), U1.B7 (D-)
- new net GND: U1.1 (EH), U1.2 (EH), U1.3 (EH), U1.4 (EH), U1.A1 (GND), U1.A12 (GND), U1.B1 (GND), U1.B12 (GND)
- no-connect marks 0 -> 2

Commit message: 5V,3.3V
Parts:
- added C1, C11, C13, C15, C17: 100nF, JLCImport:C0603, symbol JLCImport:C
- added C10: 470uF, JLCImport:MA35V470M10X13, symbol JLCImport:MA35V470M10X13
- added C12: 330uF, JLCImport:MA35V470M10X13, symbol JLCImport:MA35V470M10X13
- added C14, C16: 10uF, JLCImport:C0603, symbol JLCImport:C
- added C2, C3, C4, C5, C6, C7, C8, C9: 47uF, JLCImport:C1206, symbol JLCImport:C
- added D1: SS34, JLCImport:SS34_C7420365, symbol JLCImport:SS34_C7420365
- added L1: 100uH, JLCImport:PSPMAA1050H-101M-ANP, symbol JLCImport:PSPMAA1050H-101M-ANP
- added R1, R2: 10K, JLCImport:R0603, symbol JLCImport:R
- added U2: CH224A, JLCImport:CH224A, symbol JLCImport:CH224A
- added U3: LM2576C5-5_0, JLCImport:LM2576C5-5_0, symbol JLCImport:LM2576C5-5_0
- added U4: RT9013-33GB, JLCImport:RT9013-33GB, symbol JLCImport:RT9013-33GB
Connections:
- net +VDC: now also C1.1, C10.1, C11.2, C2.1, C3.1, C4.1, C5.1, C6.1, C7.1, C8.1, C9.1, U2.1 (VHV), U2.8 (VBUS), U3.1 (VIN)
- net CC1: now also U2.7 (CC1)
- net CC2: now also U2.6 (CC2)
- net D+: now also U2.4 (DP)
- net D-: now also U2.5 (DM)
- net GND: now also C1.2, C10.2, C11.1, C12.2, C13.1, C14.1, C15.1, C16.1, C17.1, C2.2, C3.2, C4.2, C5.2, C6.2, C7.2, C8.2, C9.2, D1.1 (A), R1.1, R2.1, U2.11 (GND), U3.3 (GND), U3.6 (GND), U4.2 (GND)
- new net: D1.2 (K), L1.1, U3.2 (OUT)
- new net: R2.2, U3.5 (ON#/OFF)
- new net: R1.2, U2.9 (CFG1)
- new net VCC3V3: C16.2, C17.2, U4.5 (VOUT)
- new net VCC5V: C12.1, C13.2, C14.2, C15.2, L1.2, U3.4 (FB), U4.1 (VIN), U4.3 (EN)
- no-connect marks 2 -> 6
Other:
- note added: "20V转5V"
- note added: "5V转3.3V"
- note added: "CH224K诱导20V"
- note added: "TYPE-C接口"
- note added: "滤波"
- moved on the sheet: U1

Commit message: 完成STM32外围电路设计
Parts:
- added C18, C19: 12pF, JLCImport:C0603, symbol JLCImport:C
- added C20, C21: 20pF, JLCImport:C0603, symbol JLCImport:C
- added C22, C24, C26: 100nF, JLCImport:C0603, symbol JLCImport:C
- added C23, C25: 10uF, JLCImport:C0603, symbol JLCImport:C
- added R3: 10K, JLCImport:R0603, symbol JLCImport:R
- added SW1: TS-1088R-02026, JLCImport:TS-1088R-02026, symbol JLCImport:TS-1088R-02026
- added U5: STM32G071CBT6, JLCImport:STM32G071CBT6, symbol JLCImport:STM32G071CBT6
- added U6: WAFER-GH1_25-4PWB, JLCImport:WAFER-GH1_25-4PWB, symbol JLCImport:WAFER-GH1_25-4PWB
- added U7: RT9013-33GB, JLCImport:RT9013-33GB, symbol JLCImport:RT9013-33GB
- added X1: X321532768KGD2SI, JLCImport:X321532768KGD2SI, symbol JLCImport:X321532768KGD2SI
- added X2: X49SM8MSD2SC, JLCImport:X49SM8MSD2SC, symbol JLCImport:X49SM8MSD2SC
Connections:
- net GND: now also C18.1, C19.1, C20.1, C21.1, C22.2, C23.1, C24.1, C25.1, C26.1, SW1.2, U5.7 (VSS/VSSA), U6.2, U6.5, U6.6, U7.2 (GND)
- net VCC3V3: now also R3.2, U5.6 (VDD/VDDA), U6.1
- net VCC5V: now also C23.2, C24.2, U7.1 (VIN), U7.3 (EN)
- new net NRST: C22.1, R3.1, SW1.1, U5.10 (PF2-NRST)
- new net OSC32_IN: C18.2, U5.2 (PC14-OSC32_IN), X1.2
- new net OSC32_OUT: C19.2, U5.3 (PC15-OSC32_OUT), X1.1
- new net OSC_IN: C20.2, U5.8 (PF0-OSC_IN), X2.2 (OSC2)
- new net OSC_OUT: C21.2, U5.9 (PF1-OSC_OUT), X2.1 (OSC1)
- new net SWCLK: U5.36 (PA14-BOOT0), U6.4
- new net SWDIO: U5.35 (PA13), U6.3
- new net VCC3V3A: C25.2, C26.2, U5.5 (VREF+), U7.5 (VOUT)
- no-connect marks 6 -> 8
Other:
- note added: "5V转模拟3.3V"
- note added: "主电源滤波"
- note removed: "滤波"

Commit message: 34
Parts:
- added C27: 470uF, JLCImport:CAP-SMD_BD10-L10.3-W10.3, symbol JLCImport:MA35V470M10X13
- added C28, C31, C33, C34: 100nF, JLCImport:C0603, symbol JLCImport:C
- added C29: 180uF, JLCImport:CAP-SMD_D6_3xL7_7, symbol JLCImport:JVJ25V180M6X8
- added C30: 4.7uF, JLCImport:C0603, symbol JLCImport:C
- added C32: 1uF, JLCImport:C0603, symbol JLCImport:C
- added D2: SS34, JLCImport:SS34_C7420365, symbol JLCImport:SS34_C7420365
- added L2: 68uH, JLCImport:IND-SMD_11_5x10_5, symbol JLCImport:SRG1040-680-M
- added R4: 1K, JLCImport:R0603, symbol JLCImport:R
- added R5, R6, R7: 10K, JLCImport:R0603, symbol JLCImport:R
- added U10: HC-PM254-5_0H-1X8PZ, JLCImport:HC-PM254-5_0H-1X8PZ, symbol JLCImport:HC-PM254-5_0H-1X8PZ
- added U8: XL1509-12E1, JLCImport:XL1509-12E1, symbol JLCImport:XL1509-12E1
- added U9: GD25Q64ESIGR, JLCImport:GD25Q64ESIGR, symbol JLCImport:GD25Q64ESIGR
- C10: footprint JLCImport:MA35V470M10X13 -> JLCImport:CAP-SMD_BD10-L10.3-W10.3
- C12: footprint JLCImport:MA35V470M10X13 -> JLCImport:CAP-SMD_D6_3xL7_7; LCSC C46550472 -> C47023104
Connections:
- net +VDC: now also C27.1, C28.2, U8.1 (VIN)
- net GND: now also C27.2, C28.1, C29.2, C30.1, C31.1, C34.2, D2.1 (A), U10.1, U8.5 (GND), U8.6 (GND), U8.7 (GND), U8.8 (GND), U9.4 (VSS)
- net VCC3V3: now also C30.2, C31.2, C34.1, R5.2, R6.1, R7.1, U10.2, U9.8 (VCC)
- net VCC3V3A: now also C32.2, C33.2
- net VCC5V: now also R4.1
- net SPI1_CS: now reaches U5.11 (PA0)
- net SPI1_CS: now also R6.2, U9.1 (CS#)
- net SPI1_SCK: now reaches U5.12 (PA1)
- net SPI1_SCK: now also U9.6 (SCLK)
- net SPI1_MOSI: now reaches U5.13 (PA2)
- net SPI1_MOSI: now also U9.5 (SI(IO0))
- net PWM1: now reaches U5.14 (PA3)
- net SPI2_MOSI: now reaches U5.15 (PA4)
- net SPI2_MOSI: now also U10.4
- net PWM2: now reaches U5.16 (PA5)
- net SPI1_MISO: now reaches U5.17 (PA6)
- net SPI1_MISO: now also U9.2 (SO(IO1))
- net PWM4: now reaches U5.22 (PB10)
- net SPI2_SCK: now reaches U5.25 (PB13)
- net SPI2_SCK: now also U10.3
- net SPI2_REST: now reaches U5.26 (PB14)
- net SPI2_REST: now also U10.5
- net SPI2_DC: now reaches U5.27 (PB15)
- net SPI2_DC: now also U10.6
- net SPI2_CS: now reaches U5.28 (PA8)
- net SPI2_CS: now also U10.7
- net USART_TX: now reaches U5.29 (PA9)
- net SPI2_CLK: now reaches U5.30 (PC6)
- net SPI2_CLK: now also U10.8
- net USART_RX: now reaches U5.32 (PA10)
- net PWM3: now reaches U5.42 (PB3)
- new net: D2.2 (K), L2.2, U8.2 (OUTPUT)
- new net: R7.2, U9.3 (WP#(IO2))
- new net: R5.1, U9.7 (HOLD#(IO3))
- new net: R4.2, U8.4 (ON/OFF)
- new net GNDA: C32.1, C33.1
- new net VCC12V: C29.1, L2.1, U8.3 (FB)
Other:
- note added: "2.0寸SPI显示器"
- note added: "20V转12 给栅极驱动供电"
- note added: "STM32系统板"
- note added: "外部FLASH"
- moved on the sheet: C10, C11, C12, C13, C14, C15, C16, C17, C18, C19, C20, C21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

Commit message: 35
Parts:
- added C35: 100nF, JLCImport:C0603, symbol JLCImport:C
- added D3: SS54, JLCImport:SS54_C22452, symbol JLCImport:SS54_C22452
- added D4: 1N5819W, JLCImport:SOD-123, symbol JLCImport:1N5819W_C963381
- added R8, R9: 5.1K, JLCImport:R0603, symbol JLCImport:R
- added U11: TYPE-C_16PLC-H10_0, JLCImport:TYPE-C_16PLC-H10_0, symbol JLCImport:TYPE-C_16PLC-H10_0
- added U12: CH340N, JLCImport:SOP-8, symbol JLCImport:CH340N_C2977777
Connections:
- net +VDC: now also D3.2 (K); no longer U1.A4 (VBUS), U1.A9 (VBUS), U1.B4 (VBUS), U1.B9 (VBUS)
- net GND: now also C35.2, R8.1, R9.2, U11.1 (EH), U11.2 (EH), U11.3 (EH), U11.4 (EH), U11.A1 (GND), U11.A12 (GND), U11.B1 (GND), U11.B12 (GND), U12.3 (GND)
- net USART_RX: now also U12.6 (TXD)
- net USART_TX: now also U12.7 (RXD)
- net VCC5V: now also D4.2 (A), U11.A4 (VBUS), U11.A9 (VBUS), U11.B4 (VBUS), U11.B9 (VBUS)
- new net: R8.2, U11.A5 (CC1)
- new net: R9.1, U11.B5 (CC2)
- new net: D3.1 (A), U1.A4 (VBUS), U1.A9 (VBUS), U1.B4 (VBUS), U1.B9 (VBUS)
- new net: D4.1 (C), U12.5 (VCC)
- new net: C35.1, U12.8 (V3)
- new net D++: U11.A6 (D+), U11.B6 (D+), U12.1 (UD+)
- new net D--: U11.A7 (D-), U11.B7 (D-), U12.2 (UD-)
- no-connect marks 8 -> 11
Other:
- note added: "2.0寸SPI显示屏"
- note added: "USART通信"
- note removed: "2.0寸SPI显示器"
